Commit message: Show sensors in rviz

File: legged_perceptive_controller/legged_perceptive/legged_perceptive_description/urdf/sensor_t265.xacro (robot description, xacro)
@@ -31,6 +31,6 @@
                 <origin xyz="0 0 0" rpy="0 0 0"/>
                 <geometry>
-                    <!-- <mesh filename="package://realsense2_description/meshes/t265.stl"/> -->
-                    <mesh filename="/home/mjw/legged_perception_control_ws/src/realsense2_description/meshes/t265.stl"/>
+                    <mesh filename="file://$(find realsense2_description)/meshes/t265.stl"/>
+                    <!-- <mesh filename="file:///home/mjw/legged_perception_control_ws/src/realsense2_description/meshes/t265.stl"/> -->
                 </geometry>
                 <material name="${name}_aluminum"/>
@@ -39,6 +39,6 @@
                 <origin xyz="0 0 0" rpy="0 0 0"/>
                 <geometry>
-                    <!-- <mesh filename="package://realsense2_description/meshes/t265.stl"/> -->
-                    <mesh filename="/home/mjw/legged_perception_control_ws/src/realsense2_description/meshes/t265.stl"/>
+                    <mesh filename="file://$(find realsense2_description)/meshes/t265.stl"/>
+                    <!-- <mesh filename="file:///home/mjw/legged_perception_control_ws/src/realsense2_description/meshes/t265.stl"/> -->
                 </geometry>
             </collision>
